File: hardware/retroduino-s1/retroduino.brd (EAGLE design)
At the start: 101.6 x 53.3 mm, 49 parts, among them IC1 25LC256-I/PT, IC2 FT232RL, IC3 AT89S8253-24JU, IC4 74HC573N, IC5 74HC157N, IC6 CY62256LL-PC, IC7 CY62256LL-PC, IC9 74LVC1G00DBV, J1 SPI_PROG_3X2, Q1 MMUN2114LT1G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

Commit message: some pcb bugs fixed:
1. !ea should be connected to vcc due to allow boot from internal flash
2. missing microcontroller gnd supply (pin 22)
Connections:
- removed net N$9: IC3.22
- net +5V: now also IC3.35
- net GND: now also IC3.22; no longer IC3.35
Routing:
- net +5V: track 366.2 -> 380.8 mm
Changed lines of the file:
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@@
 <drawing>
 <settings>
-<setting alwaysvectorfont="yes"/>
+<setting alwaysvectorfont="no"/>
 <setting verticaltext="up"/>
 </settings>
 <grid distance="50" unitdist="mil" unit="mm" style="lines" multiple="1" display="no" altdistance="5" altunitdist="mil" altunit="mm"/>
 <layers>
-<layer number="1" name="Top" color="4" fill="1" visible="no" active="yes"/>
+<layer number="1" name="Top" color="4" fill="1" visible="yes" active="yes"/>
 <layer number="16" name="Bottom" color="1" fill="1" visible="yes" active="yes"/>
 <layer number="17" name="Pads" color="2" fill="1" visible="yes" active="yes"/>
@@
 <contactref element="IC4" pad="1"/>
 <contactref element="IC5" pad="15"/>
-<contactref element="IC3" pad="35"/>
 <contactref element="C9" pad="1"/>
 <contactref element="R6" pad="1"/>
@@
 <via x="29.21" y="14.097" extent="1-16" drill="0.4"/>
 <via x="50.292" y="35.56" extent="1-16" drill="0.4"/>
+<contactref element="IC3" pad="22"/>
 </signal>
 <signal name="D7">
@@
 <wire x1="27.94" y1="29.591" x2="24.003" y2="29.591" width="1.016" layer="1"/>
 <wire x1="72.39" y1="10.16" x2="72.39" y2="5.715" width="1.016" layer="16"/>
+<contactref element="IC3" pad="35"/>
+<wire x1="40.005" y1="22.479" x2="37.846" y2="20.32" width="0.4" layer="1"/>
+<wire x1="35.56" y1="20.32" x2="37.846" y2="20.32" width="0.4" layer="1"/>
+<wire x1="40.005" y1="22.479" x2="40.005" y2="26.035" width="0.4" layer="1"/>
+<wire x1="40.005" y1="26.035" x2="40.64" y2="26.67" width="0.4" layer="1"/>
+<wire x1="43.64966875" y1="26.67" x2="44.91966875" y2="27.94" width="0.4" layer="1"/>
+<wire x1="40.64" y1="26.67" x2="43.64966875" y2="26.67" width="0.4" layer="1"/>
 </signal>
 <signal name="C_!OE">
@@
 <wire x1="20.32" y1="27.94" x2="16.422" y2="31.838" width="0.4" layer="1"/>
 <wire x1="16.422" y1="31.838" x2="16.422" y2="32.512" width="0.4" layer="1"/>
-</signal>
-<signal name="N$9">
-<contactref element="IC3" pad="22"/>
 </signal>
 <signal name="N$10">
@@
 <mfgpreviewcolor name="substratecolor" color="0xFF786E46"/>
 </mfgpreviewcolors>
-<errors>
-</errors>
 </board>
 </drawing>
