File: hardware/retroduino-s1/retroduino.sch (EAGLE design)
At the start: 49 parts, among them IC1 25LC256-I/PT, IC2 FT232RL, IC3 AT89S8253-24JU, IC4 74HC573N, IC5 74HC157N, IC6 CY62256LL-PC, IC7 CY62256LL-PC, IC9 74LVC1G00DBV, J1 SPI_PROG_3X2, Q1 MMUN2114LT1G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

Commit message: diagram and assets updated
Other:
- note added: "2018-10-28"
- note added: "8051-based Arduino-compatible microcomputer"
- note added: "Author"
- note added: "Date"
- note added: "Marcin Borowicz"
- note added: "Project"
- note added: "Retroduino-S1"
Changed lines of the file:
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@@
 <sheet>
 <plain>
+<frame x1="-185.42" y1="-45.72" x2="261.62" y2="167.64" columns="8" rows="5" layer="91"/>
+<text x="-175.26" y="-27.94" size="1.778" layer="91">Author</text>
+<text x="-175.26" y="-20.32" size="1.778" layer="91">Project</text>
+<text x="-175.26" y="-35.56" size="1.778" layer="91">Date</text>
+<text x="-162.56" y="-27.94" size="1.778" layer="91">Marcin Borowicz</text>
+<text x="-162.56" y="-20.32" size="1.778" layer="91">Retroduino-S1</text>
+<text x="-162.56" y="-35.56" size="1.778" layer="91">2018-10-28</text>
+<text x="-139.7" y="-20.32" size="1.778" layer="91">8051-based Arduino-compatible microcomputer</text>
 </plain>
 <instances>
@@
 </segment>
 </net>
+<net name="N$1" class="0">
+<segment>
+<wire x1="-177.8" y1="-38.1" x2="-177.8" y2="-30.48" width="0.1524" layer="91"/>
+<wire x1="-177.8" y1="-30.48" x2="-177.8" y2="-22.86" width="0.1524" layer="91"/>
+<wire x1="-177.8" y1="-22.86" x2="-177.8" y2="-15.24" width="0.1524" layer="91"/>
+<wire x1="-177.8" y1="-15.24" x2="-165.1" y2="-15.24" width="0.1524" layer="91"/>
+<wire x1="-165.1" y1="-15.24" x2="-142.24" y2="-15.24" width="0.1524" layer="91"/>
+<wire x1="-142.24" y1="-15.24" x2="-83.82" y2="-15.24" width="0.1524" layer="91"/>
+<wire x1="-83.82" y1="-15.24" x2="-83.82" y2="-22.86" width="0.1524" layer="91"/>
+<wire x1="-83.82" y1="-22.86" x2="-83.82" y2="-30.48" width="0.1524" layer="91"/>
+<wire x1="-83.82" y1="-30.48" x2="-83.82" y2="-38.1" width="0.1524" layer="91"/>
+<wire x1="-83.82" y1="-38.1" x2="-165.1" y2="-38.1" width="0.1524" layer="91"/>
+<wire x1="-165.1" y1="-38.1" x2="-177.8" y2="-38.1" width="0.1524" layer="91"/>
+<wire x1="-177.8" y1="-22.86" x2="-142.24" y2="-22.86" width="0.1524" layer="91"/>
+<wire x1="-142.24" y1="-22.86" x2="-83.82" y2="-22.86" width="0.1524" layer="91"/>
+<wire x1="-177.8" y1="-30.48" x2="-83.82" y2="-30.48" width="0.1524" layer="91"/>
+<wire x1="-165.1" y1="-38.1" x2="-165.1" y2="-15.24" width="0.1524" layer="91"/>
+<wire x1="-142.24" y1="-22.86" x2="-142.24" y2="-15.24" width="0.1524" layer="91"/>
+</segment>
+</net>

Commit message: dodany email na schemacie
Other:
- note added: "marcinbor85@gmail.com"
Changed lines of the file:
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@@
 <text x="-162.56" y="-35.56" size="1.778" layer="91">2018-10-28</text>
 <text x="-139.7" y="-20.32" size="1.778" layer="91">8051-based Arduino-compatible microcomputer</text>
+<text x="-139.7" y="-27.94" size="1.778" layer="91">marcinbor85@gmail.com</text>
 </plain>
 <instances>
@@
 <wire x1="-177.8" y1="-22.86" x2="-142.24" y2="-22.86" width="0.1524" layer="91"/>
 <wire x1="-142.24" y1="-22.86" x2="-83.82" y2="-22.86" width="0.1524" layer="91"/>
-<wire x1="-177.8" y1="-30.48" x2="-83.82" y2="-30.48" width="0.1524" layer="91"/>
+<wire x1="-177.8" y1="-30.48" x2="-142.24" y2="-30.48" width="0.1524" layer="91"/>
+<wire x1="-142.24" y1="-30.48" x2="-83.82" y2="-30.48" width="0.1524" layer="91"/>
 <wire x1="-165.1" y1="-38.1" x2="-165.1" y2="-15.24" width="0.1524" layer="91"/>
 <wire x1="-142.24" y1="-22.86" x2="-142.24" y2="-15.24" width="0.1524" layer="91"/>
-</segment>
-</net>
+<wire x1="-142.24" y1="-30.48" x2="-142.24" y2="-22.86" width="0.1524" layer="91"/>
+</segment>
+</net>

Commit message: some pcb bugs fixed:
1. !ea should be connected to vcc due to allow boot from internal flash
2. missing microcontroller gnd supply (pin 22)
Connections:
- removed net N$9: IC3.GND
- net +5V: now also IC3.!EA!/VPP
- net GND: now also IC3.GND; no longer IC3.!EA!/VPP
Changed lines of the file:
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@@
 <part name="GND24" library="supply1" library_urn="urn:adsk.eagle:library:371" deviceset="GND" device=""/>
 <part name="P+11" library="supply1" library_urn="urn:adsk.eagle:library:371" deviceset="+5V" device=""/>
-<part name="GND22" library="supply1" library_urn="urn:adsk.eagle:library:371" deviceset="GND" device=""/>
 <part name="GND23" library="supply1" library_urn="urn:adsk.eagle:library:371" deviceset="GND" device=""/>
 <part name="IC5" library="74xx-eu" library_urn="urn:adsk.eagle:library:85" deviceset="74*157" device="N" package3d_urn="urn:adsk.eagle:package:2009/1" technology="HC" value="74HC157N"/>
@@
 <part name="P+13" library="supply1" library_urn="urn:adsk.eagle:library:371" deviceset="+5V" device=""/>
 <part name="C15" library="rcl" library_urn="urn:adsk.eagle:library:334" deviceset="C-EU" device="C0603" package3d_urn="urn:adsk.eagle:package:23616/2" value="100n"/>
+<part name="P+22" library="supply1" library_urn="urn:adsk.eagle:library:371" deviceset="+5V" device=""/>
 </parts>
 <sheets>
@@
 <attribute name="VALUE" x="17.78" y="106.68" size="1.778" layer="96" rot="R90"/>
 </instance>
-<instance part="GND22" gate="1" x="20.32" y="45.72" smashed="yes" rot="R90">
-<attribute name="VALUE" x="20.32" y="45.72" size="1.778" layer="96"/>
-</instance>
 <instance part="GND23" gate="1" x="20.32" y="35.56" smashed="yes" rot="R90">
 <attribute name="VALUE" x="20.32" y="35.56" size="1.778" layer="96"/>
@@
 <attribute name="NAME" x="125.984" y="132.461" size="1.778" layer="95"/>
 <attribute name="VALUE" x="125.984" y="127.381" size="1.778" layer="96"/>
+</instance>
+<instance part="P+22" gate="1" x="20.32" y="45.72" smashed="yes" rot="R270">
+<attribute name="VALUE" x="20.32" y="45.72" size="1.778" layer="96"/>
 </instance>
 </instances>
@@
 <pinref part="IC4" gate="A" pin="OC"/>
 <wire x1="43.18" y1="66.04" x2="45.72" y2="66.04" width="0.1524" layer="91"/>
-</segment>
-<segment>
-<pinref part="GND22" gate="1" pin="GND"/>
-<pinref part="IC3" gate="P" pin="!EA!/VPP"/>
 </segment>
 <segment>
@@
 <wire x1="124.46" y1="119.38" x2="124.46" y2="127" width="0.1524" layer="91"/>
 </segment>
+<segment>
+<pinref part="IC3" gate="P" pin="GND"/>
+<pinref part="GND23" gate="1" pin="GND"/>
+</segment>
 </net>
 <net name="ALE" class="0">
@@
 <wire x1="45.72" y1="33.02" x2="43.18" y2="33.02" width="0.1524" layer="91"/>
 </segment>
+<segment>
+<pinref part="IC3" gate="P" pin="!EA!/VPP"/>
+<pinref part="P+22" gate="1" pin="+5V"/>
+</segment>
 </net>
 <net name="C_!OE" class="0">
@@
 </segment>
 </net>
-<net name="N$9" class="0">
-<segment>
-<pinref part="GND23" gate="1" pin="GND"/>
-<pinref part="IC3" gate="P" pin="GND"/>
-</segment>
-</net>
